Commit message: Update 2wd_properties.urdf.xacro

File: linorobot2_description/urdf/2wd_properties.urdf.xacro (robot description, xacro)
@@ -1,22 +1,22 @@
 <?xml version="1.0"?>
 <robot xmlns:xacro="http://ros.org/wiki/xacro">
-  <xacro:property name="base_length" value="0.24" />
-  <xacro:property name="base_width" value="0.275" />
-  <xacro:property name="base_height" value="0.003" />
-  <xacro:property name="base_mass" value="1" />
-  <xacro:property name="wheel_radius" value="0.045" />
-  <xacro:property name="wheel_width" value="0.01" />
-  <xacro:property name="wheel_pos_x" value="0.0" />
-  <xacro:property name="wheel_pos_y" value="0.13" />
-  <xacro:property name="wheel_pos_z" value="-0.03" />
+  <xacro:property name="base_length" value="0.27" />
+  <xacro:property name="base_width" value="0.27" />
+  <xacro:property name="base_height" value="0.150" />
+  <xacro:property name="base_mass" value="3" />
+  <xacro:property name="wheel_radius" value="0.035" />
+  <xacro:property name="wheel_width" value="0.012" />
+  <xacro:property name="wheel_pos_x" value="0.012" />
+  <xacro:property name="wheel_pos_y" value="0.100" />
+  <xacro:property name="wheel_pos_z" value="-0.06" />
   <xacro:property name="wheel_mass" value=".1" />
-  <xacro:property name="wheel_torque" value="20" />
+  <xacro:property name="wheel_torque" value="5" />
   <xacro:property name="front_caster_wheel" value="true" />
-  <xacro:property name="rear_caster_wheel" value="true" />
+  <xacro:property name="rear_caster_wheel" value="false" />
   <xacro:property name="laser_pose">
-    <origin xyz="0.12 0 0.33" rpy="0 0 0"/>
+    <origin xyz="0.060 0 0.120" rpy="0 0 0"/>
   </xacro:property>
   <xacro:property name="depth_sensor_pose">
-    <origin xyz="0.14 0.0 0.045" rpy="0 0 0"/>
+    <origin xyz="0.14 0.0 0.04" rpy="0 0 0"/>
   </xacro:property>
 </robot>

Commit message: Update 2wd_properties.urdf.xacro

File: linorobot2_description/urdf/2wd_properties.urdf.xacro (robot description, xacro)
@@ -1,22 +1,22 @@
 <?xml version="1.0"?>
 <robot xmlns:xacro="http://ros.org/wiki/xacro">
-  <xacro:property name="base_length" value="0.24" />
-  <xacro:property name="base_width" value="0.275" />
-  <xacro:property name="base_height" value="0.003" />
-  <xacro:property name="base_mass" value="1" />
-  <xacro:property name="wheel_radius" value="0.045" />
-  <xacro:property name="wheel_width" value="0.01" />
-  <xacro:property name="wheel_pos_x" value="0.0" />
-  <xacro:property name="wheel_pos_y" value="0.13" />
-  <xacro:property name="wheel_pos_z" value="-0.03" />
+  <xacro:property name="base_length" value="0.27" />
+  <xacro:property name="base_width" value="0.27" />
+  <xacro:property name="base_height" value="0.150" />
+  <xacro:property name="base_mass" value="3" />
+  <xacro:property name="wheel_radius" value="0.035" />
+  <xacro:property name="wheel_width" value="0.012" />
+  <xacro:property name="wheel_pos_x" value="0.012" />
+  <xacro:property name="wheel_pos_y" value="0.100" />
+  <xacro:property name="wheel_pos_z" value="-0.06" />
   <xacro:property name="wheel_mass" value=".1" />
-  <xacro:property name="wheel_torque" value="20" />
+  <xacro:property name="wheel_torque" value="5" />
   <xacro:property name="front_caster_wheel" value="true" />
   <xacro:property name="rear_caster_wheel" value="true" />
   <xacro:property name="laser_pose">
-    <origin xyz="0.12 0 0.33" rpy="0 0 0"/>
+    <origin xyz="-0.06 0 0.120" rpy="0 0 0"/>
   </xacro:property>
   <xacro:property name="depth_sensor_pose">
-    <origin xyz="0.14 0.0 0.045" rpy="0 0 0"/>
+    <origin xyz="0.14 0.0 0.04" rpy="0 0 0"/>
   </xacro:property>
 </robot>

Commit message: Update 2wd_properties.urdf.xacro

File: linorobot2_description/urdf/2wd_properties.urdf.xacro (robot description, xacro)
@@ -20,3 +20,6 @@
     <origin xyz="0.14 0.0 0.04" rpy="0 0 0"/>
   </xacro:property>
+  <xacro:property name="irrange_pose">
+    <origin xyz="0.13 0.0 -0.002" rpy="0 0 0"/>
+  </xacro:property>
 </robot>
