Commit message: Update irrange.urdf.xacro

File: linorobot2_description/urdf/sensors/irrange.urdf.xacro (robot description, xacro)
@@ -9,4 +9,5 @@
     </joint>
     <link name="range_link">
+      <!--
       <collision>
         <origin xyz="0 0 0" rpy="0 0 0"/>
@@ -14,5 +15,5 @@
           <box size="0.01 0.01 0.01"/>
         </geometry>
-      </collision>
+      </collision> -->
       <visual>
         <origin xyz="0 0 0" rpy="0 0 0"/>

Commit message: Update irrange.urdf.xacro

File: linorobot2_description/urdf/sensors/irrange.urdf.xacro (robot description, xacro)
@@ -5,5 +5,5 @@
       <axis xyz="0 1 0" />
       <xacro:insert_block name="origin" />
-      <parent link="base_link"/>
+      <parent link="base_footprint"/>
       <child link="range_link"/>
     </joint>
@@ -19,5 +19,5 @@
         <origin xyz="0 0 0" rpy="0 0 0"/>
         <geometry>
-          <box size="0.02 0.01 0.01"/>
+          <box size="0.015 0.01 0.10"/>
         </geometry>
       </visual>
